File: SSTC_Switch_Board/SSTC_Switch_Board.kicad_pcb (KiCad board)
At the start: 2 copper layers, 130 x 80 mm, 92 parts, among them J1 Screw_Terminal_01x02, J2 Screw_Terminal_01x02, J3 Screw_Terminal_01x02, J4 Screw_Terminal_01x02, K1 G5Q-1A4 DC12, K2 G5Q-1A4 DC12, K3 G5Q-1A4 DC12, Q1 2N3906, Q2 2N3906, Q3 2N3904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

Commit message: Audio isolator stuff and small changes
Parts:
- R18, R19, R20: footprint Resistor_THT:R_Axial_DIN0207_L6.3mm_D2.5mm_P2.54mm_Vertical -> Resistor_THT:R_Axial_DIN0207_L6.3mm_D2.5mm_P10.16mm_Horizontal
- R21, R22, R23: value 5.6k -> 10k
- moved R18 7.76 mm to (93.0, 65.7)
- moved TH1 0.90 mm to (124.6, 115.6)
- moved TH2 0.90 mm to (131.6, 115.6)
- moved R32 0.60 mm to (150.5, 61.4)
- turned R19 to 180 degrees
Routing:
- net Net-(R14-Pad2): track 59.7 -> 62.4 mm
- net +12V: track 221.4 -> 220.1 mm
- net Net-(D28-Pad2): track 7.71 -> 7.12 mm
