File: Audio_Isolator/Audio_Isolator.kicad_pcb (KiCad board)
At the start: 2 copper layers, 47 x 52 mm, 47 parts, among them J1 USB_B_Mini, J2 SJ-3523-SMT-TR, J3 SJ-3523-SMT-TR, U1 TL072, U2 TL072, U3 FODM217A, U4 FODM217A, U5 FODM217A, U6 FODM217A

Commit message: Finish Audio Isolator layout, begin routing
Parts:
- moved C1 77.8 mm to (106.0, 74.7), turned to -90 degrees
- moved C7 72.8 mm to (113.7, 87.2), turned to -90 degrees
- moved C3 69.9 mm to (109.8, 78.1), turned to 90 degrees
- moved R9 68.5 mm to (113.7, 91.1), turned to -90 degrees
- moved R4 68.4 mm to (117.3, 95.0)
- moved R10 66.7 mm to (123.3, 91.5), turned to -90 degrees
- moved C6 66.4 mm to (120.1, 84.8), turned to 180 degrees
- moved R3 65.6 mm to (106.0, 77.9), turned to -90 degrees
- moved C2 62.4 mm to (114.0, 95.0)
- moved R7 61.4 mm to (115.7, 75.0), turned to -90 degrees
- moved C10 56.8 mm to (138.9, 60.0), turned to 180 degrees
- moved R8 56.6 mm to (114.8, 78.8), turned to 180 degrees
- moved C9 54.5 mm to (135.5, 67.3)
- moved R15 52.3 mm to (133.8, 70.6), turned to -90 degrees
- moved C8 50.1 mm to (123.3, 88.5), turned to -90 degrees
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Routing:
- net -12V: track 0.00 -> 61.8 mm, vias 0 -> 6
- net +12V: track 0.00 -> 36.6 mm
- net Net-(U1-Pad2): track 0.00 -> 24.1 mm, vias 0 -> 2
- net Net-(U1-Pad1): track 0.00 -> 23.9 mm, vias 0 -> 2
- net Net-(U1-Pad5): track 0.00 -> 23.4 mm
- net Net-(U1-Pad6): track 0.00 -> 18.8 mm
- net Net-(U1-Pad7): track 0.00 -> 14.0 mm
- net Net-(U1-Pad3): track 0.00 -> 11.7 mm
- net Net-(C2-Pad1): track 0.00 -> 5.80 mm
- net Net-(J2-PadR): track 0.00 -> 4.00 mm
- net Net-(C1-Pad1): track 0.00 -> 3.70 mm
- net Net-(J2-PadT): track 0.00 -> 3.25 mm
- net Net-(R13-Pad2): track 0.00 -> 2.57 mm
- net Net-(R14-Pad2): track 0.00 -> 2.53 mm
- net Net-(R12-Pad2): track 0.00 -> 2.28 mm
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Other:
- outline, holes or cut-outs redrawn

Commit message: Files sent out for fabrication
Routing:
- net +12VA: track 0.00 -> 43.8 mm, vias 0 -> 3
- net Net-(U2-Pad6): track 0.00 -> 30.4 mm
- net -12VA: track 0.00 -> 28.7 mm, vias 0 -> 2
- net Net-(U2-Pad1): track 0.00 -> 26.2 mm, vias 0 -> 2
- net Net-(U2-Pad5): track 0.00 -> 21.5 mm
- net Net-(U2-Pad3): track 0.00 -> 17.4 mm
- net +5V: track 0.00 -> 17.3 mm
- net -12V: track 61.8 -> 66.5 mm
- net Net-(C1-Pad1): track 3.70 -> 6.21 mm
- net Net-(C1-Pad2): track 0.00 -> 1.53 mm
- net GNDD: vias 3 -> 4
- net GNDA: vias 5 -> 11
