File: SSTC_Control_Board/SSTC_Control_Board.kicad_pcb (KiCad board)
At the start: 4 copper layers, 105 x 75 mm, 149 parts, among them J1 Screw_Terminal_01x02, J2 Screw_Terminal_01x03, J3 AudioJack3, J4 Screw_Terminal_01x03, Q1 BSS84, Q2 BSS138, Q4 MMBT3906, Q5 MMBT3906, U1 ADA4891-2, U10 74HC86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

Commit message: Audio isolator stuff and small changes
Parts:
- removed D5, D6: 1N4148W, Diode_SMD:D_SOD-123
- C20: value 0.1uF -> 0.01uF
- C21: value 0.01uF -> 1000pF
- C3: value 3.3pF -> 10pF
- D3, D4: value 1N4148W -> SMAJ11CA-13-F; footprint Diode_SMD:D_SOD-123 -> Diode_SMD:D_SMA
- J3: value AudioJack3 -> SJ-3523-SMT-TR
- R39: value 100k -> 220k
- moved D4 20.1 mm to (55.0, 55.0), turned to -90 degrees
- moved C25 4.03 mm to (69.0, 64.5)
- moved R48 4.03 mm to (72.3, 64.5)
- moved R44 3.75 mm to (66.4, 63.6), turned to -90 degrees
- moved C23 3.74 mm to (64.6, 63.8), turned to -90 degrees
- moved R58 2.10 mm to (115.8, 58.6), turned to 90 degrees
- moved D3 1.69 mm to (75.5, 55.0)
- moved R43 1.12 mm to (73.5, 51.6)
- moved R42 1.07 mm to (58.7, 57.0), turned to 0 degrees
- moved C21 0.40 mm to (89.1, 72.2)
- moved R39 0.25 mm to (89.1, 75.4)
Connections:
- D3 pad 1: +5V -> GND
- D4 pad 1: Net-(C24-Pad2) -> GND
- D4 pad 2: GND -> Net-(C23-Pad2)
Routing:
- net Net-(C23-Pad2): track 9.55 -> 20.3 mm, vias 0 -> 2
- net Net-(C27-Pad2): track 12.1 -> 7.78 mm
- net Net-(D10-Pad1): track 13.2 -> 10.4 mm
- net +5V: track 75.7 -> 73.7 mm, vias 33 -> 31
- net Net-(RV1-Pad2): track 25.6 -> 27.2 mm, vias 1 -> 2
- net Net-(C24-Pad2): track 9.90 -> 8.77 mm
- net Net-(J3-PadR): track 3.50 -> 4.45 mm
- net /PLL_Block/VCO_IN: track 21.4 -> 20.5 mm, vias 0 -> 2
- net Net-(J3-PadT): track 3.35 -> 2.80 mm
- net GND: vias 187 -> 191

Commit message: Files sent out for fabrication
Parts:
- removed R44, R45: 1M, Resistor_SMD:R_0805_2012Metric
- added C34: 0.1uF, Capacitor_SMD:C_0603_1608Metric, F.Cu at (77.8, 72.5)
- added D5: LED, LED_SMD:LED_0603_1608Metric, F.Cu at (99.3, 115.0)
- added R34: 47k, Resistor_SMD:R_0805_2012Metric, F.Cu at (77.8, 69.3)
- added R35: 1k, Resistor_SMD:R_0805_2012Metric, F.Cu at (95.5, 115.0)
- C27: value 220pF -> 180pF
- C29: value 220pF -> 470pF
- J3: value SJ-3523-SMT-TR -> SJ1-3523N; footprint Connector_Audio:Jack_3.5mm_CUI_SJ-3523-SMT_Horizontal -> Repowered_Connectors:Jack_3.5mm_CUI_SJ1-3523N_Horizontal
- PS1: value IRM-03-5 -> RAC03-05SK; footprint Converter_ACDC:Converter_ACDC_MeanWell_IRM-03-xx_THT -> Repowered_Modules:RAC03-K
- R42, R43: value 100 -> 60.4
- R46, R47: value 10k -> 4.7k
- moved C23 17.1 mm to (50.8, 53.7)
- moved PS1 14.5 mm to (68.8, 107.5), turned to 0 degrees
- moved C25 14.4 mm to (56.2, 57.9), turned to 90 degrees
- moved C24 8.23 mm to (79.9, 53.7), turned to -90 degrees
- moved R42 6.82 mm to (52.8, 53.6), turned to 90 degrees
- moved R43 4.79 mm to (77.8, 53.6), turned to -90 degrees
- moved R49 3.46 mm to (77.0, 66.5), turned to 180 degrees
- moved C26 3.40 mm to (74.5, 57.9), turned to 90 degrees
- moved C27 3.00 mm to (76.0, 63.6)
- moved D4 2.73 mm to (56.2, 52.5)
- moved D3 2.71 mm to (74.5, 52.5), turned to -90 degrees
- moved J3 1.93 mm to (65.3, 49.5), turned to 180 degrees
- moved R48 0.73 mm to (73.0, 64.4)
- moved R50 0.65 mm to (77.8, 63.6)
Connections:
- J3 pad R: Net-(J3-PadR) -> Net-(C24-Pad2)
- J3 pad T: Net-(J3-PadT) -> Net-(C23-Pad2)
- PS1 pad 3: Net-(J2-Pad2) -> +5V
- R42 pad 2: Net-(J3-PadT) -> GND
- R43 pad 1: Net-(C24-Pad2) -> GND
- R43 pad 2: Net-(J3-PadR) -> Net-(C24-Pad2)
- R46 pad 1: Net-(R46-Pad1) -> Net-(C34-Pad2)
- R47 pad 2: Net-(R46-Pad1) -> Net-(C34-Pad2)
- R49 pad 1: Net-(C26-Pad1) -> Net-(R34-Pad2)
- R49 pad 2: Net-(C27-Pad2) -> Net-(C26-Pad1)
- U13 pad 3: Net-(R46-Pad1) -> Net-(R34-Pad2)
- U13 pad 5: Net-(R46-Pad1) -> Net-(C34-Pad2)
Routing:
- net Net-(J2-Pad2): track 29.0 -> 11.7 mm
- net Net-(C25-Pad1): track 1.56 -> 18.9 mm, vias 0 -> 2
- net Net-(C34-Pad2): track 0.00 -> 13.5 mm
- net Net-(R46-Pad1): track 9.37 -> 0.00 mm
- net Net-(C23-Pad2): track 20.3 -> 12.1 mm, vias 2 -> 0
- net Net-(C26-Pad1): track 1.45 -> 9.23 mm, vias 0 -> 2
- net Net-(R34-Pad2): track 0.00 -> 5.25 mm
- net Net-(J3-PadR): track 4.45 -> 0.00 mm
- net Net-(C24-Pad2): track 8.77 -> 12.2 mm
- net Net-(J3-PadT): track 2.80 -> 0.00 mm
- net Net-(D5-Pad2): track 0.00 -> 2.15 mm
- net Net-(C27-Pad1): track 7.51 -> 8.98 mm
- net +5V: track 73.7 -> 75.0 mm, vias 31 -> 32
- net Net-(C27-Pad2): track 7.78 -> 7.10 mm
- net Net-(J2-Pad3): track 18.1 -> 18.7 mm
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Other:
- outline, holes or cut-outs redrawn
- board text added: "SSTC CONTROL BOARD REV 1 (C) 2022 ADAM CORDINGLEY www.acordingley.us"
