File: SSTC_Control_Board/SSTC_Control_Board.kicad_sch (KiCad schematic)
At the start: 24 parts, among them J1 Screw_Terminal_01x02, J2 Screw_Terminal_01x03, U1 ADA4891-2, U2 74AHC1G14

Commit message: Audio isolator stuff and small changes
Parts:
- C3: value 3.3pF -> 10pF
Changed lines of the file:
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@@
     (in_bom yes) (on_board yes) (fields_autoplaced)
     (property "Reference" "C3" (id 0) (at 87.63 73.8845 90))
-    (property "Value" "3.3pF" (id 1) (at 87.63 76.6596 90))
+    (property "Value" "10pF" (id 1) (at 87.63 76.6596 90))
     (property "Footprint" "Capacitor_SMD:C_0603_1608Metric" (id 2) (at 91.44 79.0448 0)
       (effects (font (size 1.27 1.27)) hide)
@@
       (reference "#PWR057") (unit 1) (value "GND") (footprint "")
     )
-    (path "/41530295-6759-4ab0-a7bb-4c461bb04f50/e2d6a6e3-51c3-468f-8e4c-4fe80af111d0"
-      (reference "#PWR058") (unit 1) (value "+5V") (footprint "")
-    )
-    (path "/41530295-6759-4ab0-a7bb-4c461bb04f50/e6a33221-743a-42c0-9dc3-56d2ecae96a0"
-      (reference "#PWR059") (unit 1) (value "+5V") (footprint "")
-    )
     (path "/41530295-6759-4ab0-a7bb-4c461bb04f50/974e6fdc-ae5b-4364-a1bc-9c32ac7658c8"
       (reference "#PWR060") (unit 1) (value "GND") (footprint "")
@@
     )
     (path "/eb22ee3b-7b2b-4221-8133-603754bb1c0a"
-      (reference "C3") (unit 1) (value "3.3pF") (footprint "Capacitor_SMD:C_0603_1608Metric")
+      (reference "C3") (unit 1) (value "10pF") (footprint "Capacitor_SMD:C_0603_1608Metric")
     )
     (path "/fa25a430-22b0-4b1d-b9b6-dd1d8aa5ea86/213a47cd-c6b7-4a68-b67f-b376226fba3e"
@@
     )
     (path "/315e4a14-b2d5-4c23-adc3-c111b0734cac/84a68fb9-b207-458a-96c7-6e36f05c4951"
-      (reference "C20") (unit 1) (value "0.1uF") (footprint "Capacitor_SMD:C_0603_1608Metric")
+      (reference "C20") (unit 1) (value "0.01uF") (footprint "Capacitor_SMD:C_0603_1608Metric")
     )
     (path "/315e4a14-b2d5-4c23-adc3-c111b0734cac/89ee2e88-5e80-4a12-8208-11307c88501d"
-      (reference "C21") (unit 1) (value "0.01uF") (footprint "Capacitor_SMD:C_0603_1608Metric")
+      (reference "C21") (unit 1) (value "1000pF") (footprint "Capacitor_SMD:C_0603_1608Metric")
     )
     (path "/315e4a14-b2d5-4c23-adc3-c111b0734cac/2ee56d34-9923-4f5f-8038-0723bd1ed8c9"
@@
     )
     (path "/41530295-6759-4ab0-a7bb-4c461bb04f50/f96415ac-d01a-4f02-abed-a0d5e4231158"
-      (reference "C27") (unit 1) (value "220pF") (footprint "Capacitor_SMD:C_0603_1608Metric")
+      (reference "C27") (unit 1) (value "470pF") (footprint "Capacitor_SMD:C_0603_1608Metric")
     )
     (path "/41530295-6759-4ab0-a7bb-4c461bb04f50/e87c2217-57b3-492a-b2e5-24d648c43f72"
@@
     )
     (path "/41530295-6759-4ab0-a7bb-4c461bb04f50/8dbbbbb2-f812-4670-97ad-a80dc0c1bae0"
-      (reference "C29") (unit 1) (value "220pF") (footprint "Capacitor_SMD:C_0603_1608Metric")
+      (reference "C29") (unit 1) (value "470pF") (footprint "Capacitor_SMD:C_0603_1608Metric")
     )
     (path "/646d7a66-565c-4a41-a52c-4ecbd74dd2e4/d1f2f43f-31bf-4803-ab48-09b20c5b49a1"
@@
       (reference "D2") (unit 1) (value "MBR160HWTR") (footprint "Diode_SMD:D_SOD-123")
     )
-    (path "/41530295-6759-4ab0-a7bb-4c461bb04f50/58cca228-de01-4629-8de2-ae9ccc4a2836"
-      (reference "D3") (unit 1) (value "1N4148W") (footprint "Diode_SMD:D_SOD-123")
-    )
-    (path "/41530295-6759-4ab0-a7bb-4c461bb04f50/ee9c7faf-e24b-46f9-b328-6fc1ba4dcc66"
-      (reference "D4") (unit 1) (value "1N4148W") (footprint "Diode_SMD:D_SOD-123")
-    )
-    (path "/41530295-6759-4ab0-a7bb-4c461bb04f50/21413793-4245-464f-b005-42da8d56843f"
-      (reference "D5") (unit 1) (value "1N4148W") (footprint "Diode_SMD:D_SOD-123")
-    )
-    (path "/41530295-6759-4ab0-a7bb-4c461bb04f50/b7196456-4c6e-46e4-b23a-8910535134f4"
-      (reference "D6") (unit 1) (value "1N4148W") (footprint "Diode_SMD:D_SOD-123")
+    (path "/41530295-6759-4ab0-a7bb-4c461bb04f50/980a2aa2-c763-4943-8811-7049a93d6df2"
+      (reference "D3") (unit 1) (value "SMAJ11CA-13-F") (footprint "Diode_SMD:D_SMA")
+    )
+    (path "/41530295-6759-4ab0-a7bb-4c461bb04f50/55c2d721-45e2-4c18-8cef-4e3771ef0ae6"
+      (reference "D4") (unit 1) (value "SMAJ11CA-13-F") (footprint "Diode_SMD:D_SMA")
     )
     (path "/fa25a430-22b0-4b1d-b9b6-dd1d8aa5ea86/867662c0-8652-44e7-8f95-372a6456cebe"
@@
     )
     (path "/41530295-6759-4ab0-a7bb-4c461bb04f50/2a7d9994-b9e8-449d-9705-4c2a8b56bffb"
-      (reference "J3") (unit 1) (value "AudioJack3") (footprint "Connector_Audio:Jack_3.5mm_CUI_SJ-3523-SMT_Horizontal")
+      (reference "J3") (unit 1) (value "SJ-3523-SMT-TR") (footprint "Connector_Audio:Jack_3.5mm_CUI_SJ-3523-SMT_Horizontal")
     )
     (path "/646d7a66-565c-4a41-a52c-4ecbd74dd2e4/8c82293f-f721-4e91-9a44-f3a759f19b9c"
@@
     )
     (path "/315e4a14-b2d5-4c23-adc3-c111b0734cac/9999f547-bb87-4833-a606-e772a29a8545"
-      (reference "R39") (unit 1) (value "100k") (footprint "Resistor_SMD:R_0805_2012Metric")
+      (reference "R39") (unit 1) (value "220k") (footprint "Resistor_SMD:R_0805_2012Metric")
     )
     (path "/315e4a14-b2d5-4c23-adc3-c111b0734cac/a1f5d77d-bcb6-4a08-91fc-b93645459d79"
@@
     )
     (path "/41530295-6759-4ab0-a7bb-4c461bb04f50/611594dc-2210-401e-8527-f174ed894718"
-      (reference "R50") (unit 1) (value "47k") (footprint "Resistor_SMD:R_0805_2012Metric")
+      (reference "R50") (unit 1) (value "22k") (footprint "Resistor_SMD:R_0805_2012Metric")
     )
     (path "/41530295-6759-4ab0-a7bb-4c461bb04f50/b520d820-2855-440a-a2d3-147842aaf462"

Commit message: Files sent out for fabrication
Parts:
- removed PS1: IRM-03-5, Converter_ACDC:Converter_ACDC_MeanWell_IRM-03-xx_THT, symbol Converter_ACDC:IRM-03-5
- added D5: LED, LED_SMD:LED_0603_1608Metric, symbol Device:LED
- added PS1: RAC03-05SK, Repowered_Modules:RAC03-K, symbol Recom:RAC03-12SK
- added R35: 1k, Resistor_SMD:R_0805_2012Metric, symbol Device:R_US
Connections:
- net +5V: now also PS1.3 (+Vout), R35.2
- net GND: now also D5.1 (K), PS1.2 (-Vout)
- net at J2.3 (Pin_3): now also PS1.1 (AC/L)
- net at J2.2 (Pin_2): now also PS1.4 (AC/N)
- new net: D5.2 (A), R35.1
Other:
- moved on the sheet: C1, C2, C3, C40, D1, D2, J1, R1, R2, R3, R4, TP1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
