File: SSTC_Control_Board/audio.kicad_sch (KiCad schematic)
At the start: 25 parts, among them J3 AudioJack3, U13 ADA4891-2

Commit message: Audio isolator stuff and small changes
Parts:
- removed D3, D4, D5, D6: 1N4148W, Diode_SMD:D_SOD-123, symbol Diode:1N4148W
- added D3, D4: SMAJ11CA-13-F, Diode_SMD:D_SMA, symbol Device:D_TVS
- C27, C29: value 220pF -> 470pF
- J3: value AudioJack3 -> SJ-3523-SMT-TR; MFG_PN (none) -> SJ-3523-SMT-TR
- R50: value 47k -> 22k
Connections:
- net GND: now also D3.1 (A1), D4.1 (A1)
- net at C23.2, C25.2, R42.1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: now also D4.2 (A2)
- net at C24.2, C26.2, R43.1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: now also D3.2 (A2)

Commit message: Files sent out for fabrication
Parts:
- removed R44, R45: 1M, Resistor_SMD:R_0805_2012Metric, symbol Device:R_US
- added C34: 0.1uF, Capacitor_SMD:C_0603_1608Metric, symbol Device:C
- added R34: 47k, Resistor_SMD:R_0805_2012Metric, symbol Device:R_US
- C27: value 470pF -> 180pF
- J3: value SJ-3523-SMT-TR -> SJ1-3523N; footprint Connector_Audio:Jack_3.5mm_CUI_SJ-3523-SMT_Horizontal -> Repowered_Connectors:Jack_3.5mm_CUI_SJ1-3523N_Horizontal; MFG_PN SJ-3523-SMT-TR -> SJ1-3523N
- R42, R43: value 100 -> 60.4
- R46, R47: value 10k -> 4.7k
- R50: value 22k -> 47k
Connections:
- net GND: now also R42.2, R43.1, C34.1
- net at C23.2, C25.2, D4.2 (A2)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: now also J3.T
- net at C24.2, C26.2, D3.2 (A2): now also J3.R, R43.2; no longer R43.1
- net at R46.1, R47.2, U13.5 (+): now also C34.2, R34.1; no longer U13.3 (+)
- net at R49.1: now also U13.3 (+), R34.2; no longer C26.1
- net at C27.2, R48.2, R50.1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: no longer R49.2
- new net: C26.1, R49.2
Other:
- moved on the sheet: C28, J3, R42, R43, R46, R47, R49, U13C
