File: SSTC_Control_Board/pll_block.kicad_sch (KiCad schematic)
At the start: 64 parts, among them Q1 BSS84, Q2 BSS138, U14 ADA4891-2, U17 74AHC1G14, U18 TLV3501AID, U3 74HC74, U4 74HC00, U5 74AHC1G14, U6 ADA4891-2, U7 ADA4891-2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

Commit message: Files sent out for fabrication
Other:
- note removed: "DIVIDE-BY-2"
- moved on the sheet: C10, C35, C36, C37, C39, D10, D11, D8, D9, R11, R12, R13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
