File: SSTC_Control_Board/ramp_gen.kicad_sch (KiCad schematic)
At the start: 24 parts, among them Q4 MMBT3906, Q5 MMBT3906, U10 74HC86, U11 ADA4891-2, U12 ADA4891-2

Commit message: Audio isolator stuff and small changes
Parts:
- C20: value 0.1uF -> 0.01uF
- C21: value 0.01uF -> 1000pF
- R39: value 100k -> 220k
Changed lines of the file:
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@@
       (effects (font (size 1.27 1.27)) (justify right))
     )
-    (property "Value" "0.1uF" (id 1) (at 169.799 51.3966 0)
+    (property "Value" "0.01uF" (id 1) (at 169.799 51.3966 0)
       (effects (font (size 1.27 1.27)) (justify right))
     )
@@
     (in_bom yes) (on_board yes) (fields_autoplaced)
     (property "Reference" "C21" (id 0) (at 218.44 23.0845 90))
-    (property "Value" "0.01uF" (id 1) (at 218.44 25.8596 90))
+    (property "Value" "1000pF" (id 1) (at 218.44 25.8596 90))
     (property "Footprint" "Capacitor_SMD:C_0603_1608Metric" (id 2) (at 222.25 28.2448 0)
       (effects (font (size 1.27 1.27)) hide)
@@
     (in_bom yes) (on_board yes) (fields_autoplaced)
     (property "Reference" "R39" (id 0) (at 201.93 24.3545 90))
-    (property "Value" "100k" (id 1) (at 201.93 27.1296 90))
+    (property "Value" "220k" (id 1) (at 201.93 27.1296 90))
     (property "Footprint" "Resistor_SMD:R_0805_2012Metric" (id 2) (at 201.676 30.226 90)
       (effects (font (size 1.27 1.27)) hide)
