File: SSTC_Full_Bridge_Driver/SSTC_Full_Bridge_Driver.kicad_pcb (KiCad board)
At the start: 4 copper layers, 210 x 120 mm, 151 parts, among them J1 Screw_Terminal_01x04, J2 Screw_Terminal_01x03, J3 Screw_Terminal_01x03, J6 Screw_Terminal_01x03, Q1 G3R75MT12D, Q2 G3R75MT12D, Q3 G3R75MT12D, Q4 G3R75MT12D, U1 SN74LVC1G14DBV, U10 74LVC1G00, U11 74AUC1G74, U12 LMV331, U13 LMV331, U14 74LVC1G08, U15 74LVC1G08, U16 74LVC1G08, U17 74LVC1G08, U18 74LVC1G08, U19 74LVC1G08, U2 SN65HVD1050D, U20 MAX22701EASA+, U21 MAX22701EASA+, U22 MAX22701EASA+, U23 MAX22701EASA+, U3 AZ1117-3.3, U4 ISE1505A, U5 ADuM1200CR, U6 OPA333xxDBV, U7 OPA333xxDBV, U8 74LVC1G08, U9 SN74LVC1G14DBV

Commit message: Audio isolator stuff and small changes
Parts:
- U11: value 74AUC1G74 -> 74HC74; footprint Package_SO:SSOP-8_2.95x2.8mm_P0.65mm -> Package_SO:SOIC-14_3.9x8.7mm_P1.27mm
- moved R26 77.9 mm to (104.7, 87.7), turned to -90 degrees
- moved C34 76.4 mm to (108.1, 114.1)
- moved U9 74.9 mm to (100.1, 107.1), turned to 90 degrees
- moved C40 69.7 mm to (108.1, 121.2)
- moved C33 67.4 mm to (101.2, 97.5)
- moved R19 64.9 mm to (111.7, 82.5), turned to -90 degrees
- moved U10 64.4 mm to (107.8, 123.8)
- moved C28 56.4 mm to (107.7, 90.3), turned to 180 degrees
- moved C35 55.6 mm to (101.0, 121.2)
- moved R23 55.0 mm to (102.5, 87.7), turned to 90 degrees
- moved C32 49.7 mm to (97.3, 106.8), turned to 90 degrees
- moved R18 49.1 mm to (111.7, 85.9), turned to -90 degrees
- moved R17 46.3 mm to (112.6, 88.7)
- moved U8 43.7 mm to (100.7, 123.8)
- moved U15 35.9 mm to (107.8, 116.8)
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Connections:
- U11 pad 1: Net-(U11-Pad1) -> +3V3
- U11 pad 2: Net-(U11-Pad2) -> Net-(U15-Pad1)
- U11 pad 3: Net-(U11-Pad2) -> Net-(U9-Pad4)
- U11 pad 4: GND -> +3V3
- U11 pad 6: +3V3 -> Net-(U15-Pad1)
- U11 pad 7: +3V3 -> GND
- U11 pad 8: +3V3 -> unconnected-(U11-Pad8)
- U15 pad 1: Net-(U11-Pad2) -> Net-(U15-Pad1)
- U15 pad 4: /PWM_A -> /PWM_B
- U9 pad 4: Net-(U11-Pad1) -> Net-(U9-Pad4)
Routing:
- net /SHUTDOWN: track 0.00 -> 289.4 mm, vias 0 -> 6
- net +15V: track 65.5 -> 233.3 mm, vias 8 -> 7
- net /PWM_A: track 0.00 -> 161.2 mm, vias 0 -> 3
- net /SW_R: track 4.92 -> 164.2 mm, vias 1 -> 2
- net /I_SNS_L: track 0.00 -> 109.5 mm, vias 0 -> 2
- net /PWM_B: track 0.00 -> 101.6 mm, vias 0 -> 4
- net /I_SNS_R: track 0.00 -> 65.4 mm, vias 0 -> 2
- net /EN: track 0.00 -> 65.1 mm, vias 0 -> 3
- net +3V3: track 5.78 -> 67.1 mm, vias 8 -> 32
- net /PWM: track 0.00 -> 52.6 mm, vias 0 -> 4
- net /SW_L: track 35.5 -> 78.1 mm, vias 1 -> 2
- net /CS_R: track 0.00 -> 27.5 mm, vias 0 -> 4
- net /CANH: track 0.00 -> 21.3 mm
- net Net-(R17-Pad1): track 0.00 -> 19.3 mm
- net Net-(U15-Pad1): track 0.00 -> 18.0 mm
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- added copper zone on In1.Cu, net +3V3
- added copper zone on B.Cu, net GND
- added copper zone on In2.Cu, net GND
- removed copper zone on In2.Cu, net +3V3
- removed copper zone on In1.Cu, net GND

Commit message: Files sent out for fabrication
Parts:
- D5, D6: value S1MTR -> GB02SLT12-214; footprint Diode_SMD:D_SMA -> Diode_SMD:D_SMB
- PS1: value IRM-03-15 -> IRM-10-15; footprint Converter_ACDC:Converter_ACDC_MeanWell_IRM-03-xx_THT -> Converter_ACDC:Converter_ACDC_MeanWell_IRM-10-xx_THT
- moved C14 11.2 mm to (88.8, 108.3)
- moved C8 11.2 mm to (84.7, 112.4)
- moved U3 11.2 mm to (89.0, 112.4)
- moved PS1 11.0 mm to (48.4, 129.1), turned to 0 degrees
- moved D5 3.44 mm to (72.3, 69.6)
- moved D6 3.40 mm to (161.8, 69.5)
Connections:
- PS1 pad 1: Net-(J3-Pad3) -> Net-(J3-Pad2)
- PS1 pad 3: Net-(J3-Pad2) -> GND
Routing:
- net Net-(J3-Pad3): track 0.00 -> 16.6 mm
- net Net-(J3-Pad2): track 0.00 -> 16.5 mm
- net Earth: track 0.00 -> 9.34 mm
- net /EN: track 65.1 -> 70.6 mm
- net Net-(C49-Pad2): track 10.1 -> 13.2 mm
- net Net-(C51-Pad2): track 10.1 -> 13.1 mm
- net Net-(R2-Pad2): track 0.00 -> 1.67 mm
- net Net-(R1-Pad2): track 0.00 -> 1.67 mm
- net Net-(R32-Pad2): track 2.44 -> 3.97 mm
- net Net-(R33-Pad2): track 2.49 -> 3.94 mm
- net +15V: track 233.3 -> 232.6 mm
- net GND: vias 178 -> 176
Other:
- outline, holes or cut-outs redrawn
- board text added: "SSTC FULL-BRIDGE DRIVER (C) 2022 ADAM CORDINGELY www.acordingley.us"
