File: SSTC_Full_Bridge_Driver/SSTC_Full_Bridge_Driver.kicad_sch (KiCad schematic)
At the start: 151 parts, among them J1 Screw_Terminal_01x04, J2 Screw_Terminal_01x03, J3 Screw_Terminal_01x03, J6 Screw_Terminal_01x03, Q1 G3R75MT12D, Q2 G3R75MT12D, Q3 G3R75MT12D, Q4 G3R75MT12D, U1 SN74LVC1G14DBV, U10 74LVC1G00, U11 74AUC1G74, U12 LMV331, U13 LMV331, U14 74LVC1G08, U15 74LVC1G08, U16 74LVC1G08, U17 74LVC1G08, U18 74LVC1G08, U19 74LVC1G08, U2 SN65HVD1050D, U20 MAX22701EASA+, U21 MAX22701EASA+, U22 MAX22701EASA+, U23 MAX22701EASA+, U3 AZ1117-3.3, U4 ISE1505A, U5 ADuM1200CR, U6 OPA333xxDBV, U7 OPA333xxDBV, U8 74LVC1G08, U9 SN74LVC1G14DBV

Commit message: Audio isolator stuff and small changes
Parts:
- removed U11: 74AUC1G74, Package_SO:SSOP-8_2.95x2.8mm_P0.65mm, symbol 74xGxx:74AUC1G74
- added U11: 74HC74, Package_SO:SOIC-14_3.9x8.7mm_P1.27mm, symbol 74xx:74HC74
Connections:
- net +3V3: now also U11.1 (~{R}), U11.10 (~{S}), U11.13 (~{R}), U11.14 (VCC), U11.4 (~{S})
- net GND: now also U11.11 (C), U11.12 (D), U11.7 (GND)
- net PWM_A: no longer U15.4
- net PWM_B: now also U15.4
- net at U9.4: now also U11.3 (C)
- net at U15.1: now also U11.2 (D), U11.6 (~{Q})
- net at U14.2: now also U11.5 (Q)
- no-connect marks 3 -> 5
Other:
- moved on the sheet: U9

Commit message: Files sent out for fabrication
Parts:
- removed D5, D6: S1MTR, Diode_SMD:D_SMA, symbol Device:D
- removed PS1: IRM-03-15, Converter_ACDC:Converter_ACDC_MeanWell_IRM-03-xx_THT, symbol Converter_ACDC:IRM-03-15
- added D5, D6: GB02SLT12-214, Diode_SMD:D_SMB, symbol Device:D_Schottky
- added PS1: IRM-10-15, Converter_ACDC:Converter_ACDC_MeanWell_IRM-10-xx_THT, symbol Converter_ACDC:IRM-10-15
Connections:
- net +15V: now also PS1.4 (+Vo)
- net GND: now also PS1.3 (-Vo)
- net at C49.2, C53.2, C55.2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: now also D5.1 (K)
- net at C51.2, C54.2, C56.2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: now also D6.1 (K)
- net at J3.3 (Pin_3): now also PS1.2 (AC/L)
- net at J3.2 (Pin_2): now also PS1.1 (AC/N)
- net at R32.2: now also D5.2 (A)
- net at R33.2: now also D6.2 (A)
Other:
- note added: "15V is 670mA capable"
- note removed: "15V is 200mA capable"
Changed lines of the file:
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@@
     (effects (font (size 1.5 1.5)) (justify right bottom))
   )
-  (text "15V is 200mA capable" (at 105.41 29.21 180)
+  (text "15V is 670mA capable" (at 105.41 29.21 180)
     (effects (font (size 1.5 1.5)) (justify right bottom))
   )
@@
   (symbol (lib_id "Device:Q_NMOS_GDS") (at 391.16 157.48 0) (unit 1)
     (in_bom yes) (on_board yes) (fields_autoplaced)
-    (property "Reference" "Q3" (id 0) (at 396.367 156.5715 0)
+    (property "Reference" "Q3" (id 0) (at 396.367 156.6453 0)
       (effects (font (size 1.27 1.27)) (justify left))
     )
-    (property "Value" "G3R75MT12D" (id 1) (at 396.367 159.3466 0)
+    (property "Value" "G3R75MT12D" (id 1) (at 396.367 159.1822 0)
       (effects (font (size 1.27 1.27)) (justify left))
     )
@@
     (pin "2")
   )
-  (symbol (lib_id "Converter_ACDC:IRM-03-15") (at 76.2 43.18 0) (unit 1)
-    (in_bom yes) (on_board yes) (fields_autoplaced)
-    (property "Reference" "PS1" (id 0) (at 76.2 34.1335 0))
-    (property "Value" "IRM-03-15" (id 1) (at 76.2 36.9086 0))
-    (property "Footprint" "Converter_ACDC:Converter_ACDC_MeanWell_IRM-03-xx_THT" (id 2) (at 76.2 52.07 0)
-      (effects (font (size 1.27 1.27)) hide)
-    )
-    (property "Datasheet" "https://www.meanwell.com/Upload/PDF/IRM-03/IRM-03-SPEC.PDF" (id 3) (at 76.2 53.34 0)
-      (effects (font (size 1.27 1.27)) hide)
-    )
-    (pin "1")
-    (pin "14")
-    (pin "16")
-    (pin "3")
-    (pin "5")
-  )
   (symbol (lib_id "Device:C") (at 214.63 217.17 0) (mirror x) (unit 1)
     (in_bom yes) (on_board yes)
@@
       (effects (font (size 1.27 1.27)) hide)
     )
+    (pin "1")
+    (pin "2")
+    (pin "3")
+    (pin "4")
+    (pin "5")
+    (pin "6")
     (pin "10")
     (pin "11")
@@
     (pin "8")
     (pin "9")
+    (pin "14")
+    (pin "7")
   )
   (symbol (lib_id "Device:R_US") (at 184.15 60.96 270) (mirror x) (unit 1)
@@
     (pin "1")
   )
+  (symbol (lib_id "Device:D_Schottky") (at 345.44 24.13 180) (unit 1)
+    (in_bom yes) (on_board yes) (fields_autoplaced)
+    (property "Reference" "D5" (id 0) (at 345.7575 19.1602 0))
+    (property "Value" "GB02SLT12-214" (id 1) (at 345.7575 21.6971 0))
+    (property "Footprint" "Diode_SMD:D_SMB" (id 2) (at 345.44 24.13 0)
+      (effects (font (size 1.27 1.27)) hide)
+    )
+    (property "Datasheet" "~" (id 3) (at 345.44 24.13 0)
+      (effects (font (size 1.27 1.27)) hide)
+    )
+    (pin "1")
+    (pin "2")
+  )
   (symbol (lib_id "power:GNDA") (at 102.87 143.51 0) (unit 1)
     (in_bom yes) (on_board yes) (fields_autoplaced)
@@
     (pin "1")
   )
-  (symbol (lib_id "Device:D") (at 345.44 24.13 180) (unit 1)
-    (in_bom yes) (on_board yes) (fields_autoplaced)
-    (property "Reference" "D5" (id 0) (at 345.44 18.8935 0))
-    (property "Value" "S1MTR" (id 1) (at 345.44 21.6686 0))
-    (property "Footprint" "Diode_SMD:D_SMA" (id 2) (at 345.44 24.13 0)
-      (effects (font (size 1.27 1.27)) hide)
-    )
-    (property "Datasheet" "~" (id 3) (at 345.44 24.13 0)
-      (effects (font (size 1.27 1.27)) hide)
-    )
-    (pin "1")
-    (pin "2")
-  )
   (symbol (lib_id "Device:R_US") (at 224.79 207.01 0) (mirror x) (unit 1)
     (in_bom yes) (on_board yes) (fields_autoplaced)
@@
       (effects (font (size 1.27 1.27)) hide)
     )
+    (pin "1")
+    (pin "2")
+    (pin "3")
+    (pin "4")
+    (pin "5")
+    (pin "6")
+    (pin "10")
+    (pin "11")
+    (pin "12")
+    (pin "13")
+    (pin "8")
+    (pin "9")
     (pin "14")
     (pin "7")
@@
     (pin "2")
   )
-  (symbol (lib_id "Device:D") (at 345.44 142.24 180) (unit 1)
-    (in_bom yes) (on_board yes) (fields_autoplaced)
-    (property "Reference" "D6" (id 0) (at 345.44 137.0035 0))
-    (property "Value" "S1MTR" (id 1) (at 345.44 139.7786 0))
-    (property "Footprint" "Diode_SMD:D_SMA" (id 2) (at 345.44 142.24 0)
-      (effects (font (size 1.27 1.27)) hide)
-    )
-    (property "Datasheet" "~" (id 3) (at 345.44 142.24 0)
-      (effects (font (size 1.27 1.27)) hide)
-    )
-    (pin "1")
-    (pin "2")
-  )
   (symbol (lib_id "Device:C") (at 97.79 142.24 90) (unit 1)
     (in_bom yes) (on_board yes) (fields_autoplaced)
@@
     (pin "1")
   )
+  (symbol (lib_id "Converter_ACDC:IRM-10-15") (at 76.2 43.18 0) (unit 1)
+    (in_bom yes) (on_board yes) (fields_autoplaced)
+    (property "Reference" "PS1" (id 0) (at 76.2 34.4002 0))
+    (property "Value" "IRM-10-15" (id 1) (at 76.2 36.9371 0))
+    (property "Footprint" "Converter_ACDC:Converter_ACDC_MeanWell_IRM-10-xx_THT" (id 2) (at 76.2 52.07 0)
+      (effects (font (size 1.27 1.27)) hide)
+    )
+    (property "Datasheet" "https://www.meanwell.com/Upload/PDF/IRM-10/IRM-10-SPEC.PDF" (id 3) (at 76.2 53.34 0)
+      (effects (font (size 1.27 1.27)) hide)
+    )
+    (pin "1")
+    (pin "2")
+    (pin "3")
+    (pin "4")
+  )
   (symbol (lib_id "Device:C") (at 293.37 212.09 0) (mirror x) (unit 1)
     (in_bom yes) (on_board yes) (fields_autoplaced)
@@
     (pin "5")
     (pin "6")
+    (pin "10")
+    (pin "11")
+    (pin "12")
+    (pin "13")
+    (pin "8")
+    (pin "9")
+    (pin "14")
+    (pin "7")
   )
   (symbol (lib_id "Connector:Screw_Terminal_01x03") (at 46.99 43.18 180) (unit 1)
@@
     (pin "1")
   )
+  (symbol (lib_id "Device:D_Schottky") (at 345.44 142.24 180) (unit 1)
+    (in_bom yes) (on_board yes) (fields_autoplaced)
+    (property "Reference" "D6" (id 0) (at 345.7575 137.2702 0))
+    (property "Value" "GB02SLT12-214" (id 1) (at 345.7575 139.8071 0))
+    (property "Footprint" "Diode_SMD:D_SMB" (id 2) (at 345.44 142.24 0)
+      (effects (font (size 1.27 1.27)) hide)
+    )
+    (property "Datasheet" "~" (id 3) (at 345.44 142.24 0)
+      (effects (font (size 1.27 1.27)) hide)
+    )
+    (pin "1")
+    (pin "2")
+  )
   (symbol (lib_id "power:GNDA") (at 92.71 161.29 0) (unit 1)
     (in_bom yes) (on_board yes) (fields_autoplaced)
@@
       (reference "D4") (unit 1) (value "LED") (footprint "LED_SMD:LED_0603_1608Metric")
     )
-    (path "/7557ab4d-3de1-4508-abec-6100977ea968"
-      (reference "D5") (unit 1) (value "S1MTR") (footprint "Diode_SMD:D_SMA")
+    (path "/5aeb74e4-735d-45ad-a228-3961c3ba65cf"
+      (reference "D5") (unit 1) (value "GB02SLT12-214") (footprint "Diode_SMD:D_SMB")
     )
-    (path "/b9a31def-9264-403e-96be-22eca948736a"
-      (reference "D6") (unit 1) (value "S1MTR") (footprint "Diode_SMD:D_SMA")
+    (path "/f2ae6f35-b5fc-461f-8e79-acc33ea137e5"
+      (reference "D6") (unit 1) (value "GB02SLT12-214") (footprint "Diode_SMD:D_SMB")
     )
     (path "/5781698f-0bbd-4c2e-87ff-ff97378ab476"
@@
       (reference "NT3") (unit 1) (value "NetTie_2") (footprint "NetTie:NetTie-2_SMD_Pad0.5mm")
     )
-    (path "/46383ef7-67ba-4d8a-883b-0481e677c870"
-      (reference "PS1") (unit 1) (value "IRM-03-15") (footprint "Converter_ACDC:Converter_ACDC_MeanWell_IRM-03-xx_THT")
+    (path "/baf2597e-ea0d-47b4-8341-401cefaf0e49"
+      (reference "PS1") (unit 1) (value "IRM-10-15") (footprint "Converter_ACDC:Converter_ACDC_MeanWell_IRM-10-xx_THT")
     )
     (path "/11462ed2-ae29-49a7-b71b-2dc8d37e56a6"
