File: SSTC_PFC_Power_Supply/SSTC_PFC_Power_Supply.kicad_pcb (KiCad board)
At the start: 2 copper layers, 165 x 110 mm, 62 parts, among them J1 1766246, J2 1766246, Q1 G3R75MT12D, U1 ICE2PCS01, U2 1ED44175N01B

Commit message: Audio isolator stuff and small changes
Parts:
- moved D3 1.60 mm to (117.1, 125.5)
Routing:
- net /VOUT: track 60.0 -> 58.0 mm
Changed lines of the file:
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@@
   )
   (footprint "Diode_SMD:D_SMC" (layer "F.Cu")
-    (at 115.5 125.5 90)
+    (at 117.1 125.55 90)
     (descr "Diode SMC (DO-214AB)")
     (tags "Diode SMC (DO-214AB)")
@@
   (segment (start 146.6375 65.7) (end 146.6375 67.5) (width 0.5) (layer "F.Cu") (net 12))
   (segment (start 150.195 51.05) (end 150.195 58.15) (width 0.5) (layer "F.Cu") (net 12))
-  (via (at 116.65 120.4) (size 0.8) (drill 0.4) (layers "F.Cu" "B.Cu") (net 13))
-  (via (at 114.45 120.4) (size 0.8) (drill 0.4) (layers "F.Cu" "B.Cu") (net 13))
-  (via (at 115.55 120.4) (size 0.8) (drill 0.4) (layers "F.Cu" "B.Cu") (net 13))
+  (via (at 118.25 120.45) (size 0.8) (drill 0.4) (layers "F.Cu" "B.Cu") (net 13))
+  (via (at 116.05 120.45) (size 0.8) (drill 0.4) (layers "F.Cu" "B.Cu") (net 13))
+  (via (at 117.15 120.45) (size 0.8) (drill 0.4) (layers "F.Cu" "B.Cu") (net 13))
   (via (at 105.9 121.2) (size 1.6) (drill 1) (layers "F.Cu" "B.Cu") (net 13))
   (segment (start 79.95 124.55) (end 92.15 124.55) (width 3) (layer "B.Cu") (net 13))
@@
   (segment (start 121.55 67.4) (end 136.5 52.45) (width 0.35) (layer "F.Cu") (net 14))
   (segment (start 136.5 52.45) (end 138.1325 52.45) (width 0.35) (layer "F.Cu") (net 14))
-  (segment (start 118 131.4) (end 163.28 131.4) (width 2) (layer "F.Cu") (net 15))
-  (segment (start 115.5 128.9) (end 118 131.4) (width 2) (layer "F.Cu") (net 15))
   (segment (start 163.28 131.4) (end 167.78 126.9) (width 2) (layer "F.Cu") (net 15))
+  (segment (start 119.9 131.4) (end 163.28 131.4) (width 2) (layer "F.Cu") (net 15))
+  (segment (start 117.45 128.95) (end 119.9 131.4) (width 2) (layer "F.Cu") (net 15))
   (segment (start 198.5 49.1625) (end 198.5 54) (width 0.35) (layer "F.Cu") (net 15))
   (via (at 170.75 128.45) (size 0.8) (drill 0.4) (layers "F.Cu" "B.Cu") (net 15))
@@
     (connect_pads thru_hole_only (clearance 0.508))
     (min_thickness 0.254) (filled_areas_thickness no)
-    (fill yes (thermal_gap 0.35) (thermal_bridge_width 0.35))
+    (fill yes (thermal_gap 0.4) (thermal_bridge_width 0.5))
     (polygon
       (pts
@@
       (pts
         (xy 195.9 62.3)
-        (xy 200.7 67.1)
-        (xy 200.7 113)
-        (xy 185.3 113)
-        (xy 185.3 57.8)
+        (xy 200.45 67.1)
+        (xy 200.45 113)
+        (xy 185.65 113)
+        (xy 185.65 57.8)
         (xy 195.9 57.8)
       )
@@
         (xy 169.2 118)
         (xy 200.45 118)
-        (xy 203.95 114.55)
-        (xy 203.95 65.45)
+        (xy 204.1 114.4)
+        (xy 204.1 65.6)
         (xy 200 61.5)
         (xy 200 58)
@@
     (polygon
       (pts
-        (xy 129 123.4)
+        (xy 129.5 123.4)
         (xy 103.9 123.4)
         (xy 103.9 112)
-        (xy 129 112)
+        (xy 129.5 112)
       )
     )
@@
         (xy 169.2 118)
         (xy 200.5 118)
-        (xy 203.95 114.55)
-        (xy 203.95 55)
+        (xy 204.1 114.55)
+        (xy 204.1 55)
         (xy 212 55)
       )

Commit message: Files sent out for fabrication
Parts:
- PS1: value IRM-02-15S -> IRM-02-15; footprint Converter_ACDC:Converter_ACDC_MeanWell_IRM-02-xx_SMD -> Converter_ACDC:Converter_ACDC_MeanWell_IRM-02-xx_THT
- moved PS1 19.2 mm to (93.0, 30.8), turned to 0 degrees
Connections:
- PS1 pad 1: /LIVE_FUSED -> /NEUTRAL
- PS1 pad 3: (no net) -> GND
Routing:
- net /LIVE_FUSED: track 39.2 -> 43.8 mm
- net /VOUT: track 58.0 -> 56.4 mm
- net +15V: track 60.7 -> 62.1 mm
- net GND: vias 33 -> 30
