File: SSTC_PFC_Power_Supply/SSTC_PFC_Power_Supply.kicad_sch (KiCad schematic)
At the start: 62 parts, among them J1 1766246, J2 1766246, Q1 G3R75MT12D, U1 ICE2PCS01, U2 1ED44175N01B

Commit message: Files sent out for fabrication
Parts:
- removed PS1: IRM-02-15S, Converter_ACDC:Converter_ACDC_MeanWell_IRM-02-xx_SMD, symbol Converter_ACDC:IRM-02-15S
- added PS1: IRM-02-15, Converter_ACDC:Converter_ACDC_MeanWell_IRM-02-xx_THT, symbol Converter_ACDC:IRM-02-15
Connections:
- net +15V: now also PS1.4 (+Vo)
- net GND: now also PS1.3 (-Vo)
- net LIVE_FUSED: now also PS1.2 (AC/L)
- net NEUTRAL: now also PS1.1 (AC/N)
Changed lines of the file:
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@@
     (stroke (width 0) (type default) (color 0 0 0 0))
   )
-  (wire (pts (xy 152.4 128.27) (xy 160.02 128.27))
+  (wire (pts (xy 152.4 130.81) (xy 160.02 130.81))
     (stroke (width 0) (type default) (color 0 0 0 0))
   )
@@
     (stroke (width 0) (type default) (color 0 0 0 0))
   )
-  (wire (pts (xy 152.4 128.27) (xy 152.4 135.89))
+  (wire (pts (xy 152.4 130.81) (xy 152.4 135.89))
     (stroke (width 0) (type default) (color 0 0 0 0))
   )
@@
     (stroke (width 0) (type default) (color 0 0 0 0))
   )
-  (wire (pts (xy 160.02 128.27) (xy 160.02 118.11))
+  (wire (pts (xy 160.02 130.81) (xy 160.02 118.11))
     (stroke (width 0) (type default) (color 0 0 0 0))
   )
@@
     )
     (pin "1")
-  )
-  (symbol (lib_id "Converter_ACDC:IRM-02-15S") (at 64.77 100.33 0) (unit 1)
-    (in_bom yes) (on_board yes) (fields_autoplaced)
-    (property "Reference" "PS1" (id 0) (at 64.77 92.5535 0))
-    (property "Value" "IRM-02-15S" (id 1) (at 64.77 95.3286 0))
-    (property "Footprint" "Converter_ACDC:Converter_ACDC_MeanWell_IRM-02-xx_SMD" (id 2) (at 64.77 107.95 0)
-      (effects (font (size 1.27 1.27)) hide)
-    )
-    (property "Datasheet" "https://www.meanwell.com/Upload/PDF/IRM-02/IRM-02-SPEC.PDF" (id 3) (at 64.77 100.33 0)
-      (effects (font (size 1.27 1.27)) hide)
-    )
-    (pin "1")
-    (pin "12")
-    (pin "13")
-    (pin "24")
   )
   (symbol (lib_id "Device:C") (at 111.76 58.42 0) (unit 1)
@@
     )
   )
+  (symbol (lib_id "Converter_ACDC:IRM-02-15") (at 64.77 100.33 0) (unit 1)
+    (in_bom yes) (on_board yes) (fields_autoplaced)
+    (property "Reference" "PS1" (id 0) (at 64.77 92.8202 0))
+    (property "Value" "IRM-02-15" (id 1) (at 64.77 95.3571 0))
+    (property "Footprint" "Converter_ACDC:Converter_ACDC_MeanWell_IRM-02-xx_THT" (id 2) (at 64.77 107.95 0)
+      (effects (font (size 1.27 1.27)) hide)
+    )
+    (property "Datasheet" "https://www.meanwell.com/Upload/PDF/IRM-02/IRM-02-SPEC.PDF" (id 3) (at 74.93 109.22 0)
+      (effects (font (size 1.27 1.27)) hide)
+    )
+    (pin "1")
+    (pin "2")
+    (pin "3")
+    (pin "4")
+  )
   (symbol (lib_id "Device:R_US") (at 217.17 80.01 180) (unit 1)
     (in_bom yes) (on_board yes) (fields_autoplaced)
@@
       (reference "L3") (unit 1) (value "100uH") (footprint "Repowered_Inductors_THT:L_Bourns_1140-101K-RC")
     )
-    (path "/3247fd9c-2a54-4b0f-b2d3-c8291d505bfb"
-      (reference "PS1") (unit 1) (value "IRM-02-15S") (footprint "Converter_ACDC:Converter_ACDC_MeanWell_IRM-02-xx_SMD")
+    (path "/7ee6df27-950a-4e3b-95d5-b0cae8311659"
+      (reference "PS1") (unit 1) (value "IRM-02-15") (footprint "Converter_ACDC:Converter_ACDC_MeanWell_IRM-02-xx_THT")
     )
     (path "/88b00517-35e2-436e-b4f9-6cc3e15d0799"
